File: CM4_HighSpeed.kicad_sch (KiCad schematic)
At the start: 5 parts, among them J6 690-019-298-412, U1 RT9742SNGV

Commit message: worked some more on converting components (unfinished)
Parts:
- added J9: HDMI_E, symbol Connector:HDMI_E
Connections:
- net GND: now also J9.11 (CKS), J9.17 (GND), J9.2 (D2S), J9.5 (D1S), J9.8 (D0S), J9.SH
- net HDMI0_CEC: now also J9.13 (CEC)
- net HDMI0_CK_N: now also J9.12 (CK-)
- net HDMI0_CK_P: now also J9.10 (CK+)
- net HDMI0_D0_N: now also J9.9 (D0-)
- net HDMI0_D0_P: now also J9.7 (D0+)
- net HDMI0_D1_N: now also J9.6 (D1-)
- net HDMI0_D1_P: now also J9.4 (D1+)
- net HDMI0_D2_N: now also J9.3 (D2-)
- net HDMI0_D2_P: now also J9.1 (D2+)
- net HDMI0_HOTPLUG: now also J9.19 (HPD)
- net HDMI0_SCL: now also J9.15 (SCL)
- net HDMI0_SDA: now also J9.16 (SDA)
- net HDMI_5v: now also J9.18 (+5V)
- no-connect marks 3 -> 4
