File: CM4_GPIO.kicad_sch (KiCad schematic)
At the start: 21 parts, among them J3 Conn_01x03, J4 THD-20-R, SW2 SW_Push, U2 74LVC1G07SE-7, U3 74LVC1G07SE-7, U8 74AUC1G07

Commit message: random stuff before i screw with my windows install
Connections:
- net +3.3V_PWR: no longer D2.2 (A), U3.5 (VCC)
- new net +3.3V_PWR_1: D2.2 (A), U3.5 (VCC)
- no-connect marks 30 -> 31
Other:
- note added: "Each 3.3V can support 300mA"
Changed lines of the file:
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@@
 	)
 	(junction
+		(at 45.72 124.46)
+		(diameter 0)
+		(color 0 0 0 0)
+	)
+	(junction
 		(at 198.12 104.14)
 		(diameter 0)
@@
 	)
 	(junction
+		(at 40.64 124.46)
+		(diameter 0)
+		(color 0 0 0 0)
+	)
+	(junction
 		(at 187.96 111.76)
 		(diameter 0)
@@
 	)
 	(junction
-		(at 40.64 127)
-		(diameter 0)
-		(color 0 0 0 0)
-	)
-	(junction
 		(at 107.95 86.36)
 		(diameter 0)
@@
 	)
 	(junction
-		(at 40.64 124.46)
-		(diameter 0)
-		(color 0 0 0 0)
-	)
-	(junction
 		(at 213.36 43.18)
 		(diameter 1.016)
@@
 	)
 	(junction
-		(at 34.29 127)
-		(diameter 0)
-		(color 0 0 0 0)
-	)
-	(junction
 		(at 107.95 35.56)
 		(diameter 0)
@@
 	)
 	(no_connect
+		(at 106.68 114.3)
+	)
+	(no_connect
 		(at 45.72 137.16)
 	)
@@
 	(wire
 		(pts
-			(xy 27.94 127) (xy 34.29 127)
-		)
-		(stroke
-			(width 0)
-			(type default)
-		)
-	)
-	(wire
-		(pts
 			(xy 106.68 27.94) (xy 107.95 27.94)
 		)
@@
 	(wire
 		(pts
-			(xy 40.64 127) (xy 45.72 127)
-		)
-		(stroke
-			(width 0)
-			(type default)
-		)
-	)
-	(wire
-		(pts
 			(xy 106.68 134.62) (xy 107.95 134.62)
 		)
@@
 	(wire
 		(pts
-			(xy 212.09 30.48) (xy 213.36 30.48)
+			(xy 27.94 124.46) (xy 40.64 124.46)
 		)
 		(stroke
 			(width 0)
-			(type solid)
+			(type default)
 		)
 	)
 	(wire
 		(pts
-			(xy 27.94 119.38) (xy 45.72 119.38)
+			(xy 212.09 30.48) (xy 213.36 30.48)
 		)
 		(stroke
@@
 	(wire
 		(pts
-			(xy 144.78 123.19) (xy 146.05 123.19)
+			(xy 27.94 119.38) (xy 45.72 119.38)
 		)
 		(stroke
 			(width 0)
-			(type default)
+			(type solid)
 		)
 	)
 	(wire
 		(pts
-			(xy 34.29 127) (xy 40.64 127)
+			(xy 144.78 123.19) (xy 146.05 123.19)
 		)
 		(stroke
@@
 	(wire
 		(pts
+			(xy 45.72 124.46) (xy 45.72 127)
+		)
+		(stroke
+			(width 0)
+			(type default)
+		)
+	)
+	(wire
+		(pts
 			(xy 198.12 76.2) (xy 199.39 76.2)
 		)
@@
 	(wire
 		(pts
-			(xy 40.64 124.46) (xy 40.64 127)
-		)
-		(stroke
-			(width 0)
-			(type default)
-		)
-	)
-	(wire
-		(pts
 			(xy 44.45 93.98) (xy 45.72 93.98)
 		)
@@
 		)
 	)
+	(text "Each 3.3V \ncan support \n300mA"
+		(exclude_from_sim no)
+		(at 21.844 129.54 0)
+		(effects
+			(font
+				(size 1.27 1.27)
+			)
+		)
+	)
 	(text "40Way GPIO Header"
 		(exclude_from_sim no)
@@
 		)
 	)
-	(hierarchical_label "+3.3V_PWR"
-		(shape input)
-		(at 140.97 165.1 90)
+	(hierarchical_label "ID_SC"
+		(shape output)
+		(at 124.46 63.5 0)
 		(fields_autoplaced yes)
 		(effects
@@
 		)
 	)
-	(hierarchical_label "ID_SC"
-		(shape output)
-		(at 124.46 63.5 0)
+	(hierarchical_label "CAN_SPI_MISO"
+		(shape input)
+		(at 27.94 68.58 180)
 		(fields_autoplaced yes)
 		(effects
@@
 				(size 1.27 1.27)
 			)
-			(justify left)
+			(justify right)
 		)
 	)
-	(hierarchical_label "CAN_SPI_MISO"
-		(shape input)
-		(at 27.94 68.58 180)
+	(hierarchical_label "+3.3V_PWR"
+		(shape output)
+		(at 27.94 124.46 180)
 		(fields_autoplaced yes)
 		(effects
@@
 		)
 	)
-	(hierarchical_label "CAN_SPI_MOSI"
-		(shape output)
-		(at 27.94 73.66 180)
+	(hierarchical_label "+3.3V_PWR_1"
+		(shape input)
+		(at 140.97 165.1 90)
 		(fields_autoplaced yes)
 		(effects
@@
 				(size 1.27 1.27)
 			)
-			(justify right)
+			(justify left)
 		)
 	)
-	(hierarchical_label "CAN_SPI_CS"
+	(hierarchical_label "CAN_SPI_MOSI"
 		(shape output)
-		(at 124.46 68.58 0)
+		(at 27.94 73.66 180)
 		(fields_autoplaced yes)
 		(effects
@@
 				(size 1.27 1.27)
 			)
-			(justify left)
+			(justify right)
 		)
 	)
-	(hierarchical_label "+3.3V_PWR"
-		(shape input)
-		(at 157.48 147.32 90)
+	(hierarchical_label "CAN_SPI_CS"
+		(shape output)
+		(at 124.46 68.58 0)
 		(fields_autoplaced yes)
 		(effects
@@
 		)
 	)
-	(hierarchical_label "+3.3V_PWR"
-		(shape output)
-		(at 27.94 127 180)
+	(hierarchical_label "GLOBAL_EN"
+		(shape input)
+		(at 124.46 144.78 0)
 		(fields_autoplaced yes)
 		(effects
@@
 				(size 1.27 1.27)
 			)
-			(justify right)
+			(justify left)
 		)
 	)
-	(hierarchical_label "GLOBAL_EN"
+	(hierarchical_label "+3.3V_PWR_1"
 		(shape input)
-		(at 124.46 144.78 0)
+		(at 157.48 147.32 90)
 		(fields_autoplaced yes)
 		(effects
@@
 					(unit 1)
 				)
-			)
-		)
-	)
-	(symbol
-		(lib_id "power:PWR_FLAG")
-		(at 34.29 127 0)
-		(unit 1)
-		(exclude_from_sim no)
-		(in_bom yes)
-		(on_board yes)
-		(dnp no)
-		(property "Reference" "#FLG04"
-			(at 34.29 125.095 0)
-			(effects
-				(font
-					(size 1.27 1.27)
-				)
-				(hide yes)
-			)
-		)
-		(property "Value" "PWR_FLAG"
-			(at 34.798 128.524 0)
-			(effects
-				(font
-					(size 1.27 1.27)
-				)
-			)
-		)
-		(property "Footprint" ""
-			(at 34.29 127 0)
-			(effects
-				(font
-					(size 1.27 1.27)
-				)
-				(hide yes)
-			)
-		)
-		(property "Datasheet" "~"
-			(at 34.29 127 0)
-			(effects
-				(font
-					(size 1.27 1.27)
-				)
-				(hide yes)
-			)
-		)
-		(property "Description" "Special symbol for telling ERC where power comes from"
-			(at 34.29 127 0)
-			(effects
-				(font
-					(size 1.27 1.27)
-				)
-				(hide yes)
-			)
-		)
-		(pin "1"
-		)
-		(instances
-			(project ""
-				(path "/e4d65698-b8ec-4bf6-9f2b-a5010377155a/353ee88d-a044-4c9d-80a8-948975426026"
-					(reference "#FLG04")
-					(unit 1)
-				)

Commit message: we ballin??
Parts:
- removed J3: Conn_01x03, Connector_PinHeader_2.54mm:PinHeader_1x03_P2.54mm_Vertical, symbol Connector_Generic:Conn_01x03
- removed J4: THD-20-R, Connector_PinHeader_2.54mm:PinHeader_2x20_P2.54mm_Vertical, symbol Connector_Generic:Conn_02x20_Odd_Even
- removed Module2: ComputeModule4-CM4, CM4IO:Raspberry-Pi-4-Compute-Module, symbol CM4IO:ComputeModule4-CM4
- removed U2, U3: 74LVC1G07SE-7, Package_TO_SOT_SMD:SOT-353_SC-70-5, symbol CM4IO:74LVC1G07_copy
- removed U8: 74AUC1G07, symbol 74xGxx:74AUC1G07
- added IC5: 74LVC1G07QSE-7, SOT65P210X110-5N, symbol 74LVC1G07QSE-7:74LVC1G07QSE-7
- added J3: THD-20-R, Connector_PinHeader_2.54mm:PinHeader_2x20_P2.54mm_Vertical, symbol Connector_Generic:Conn_02x20_Odd_Even
- added Module1: ComputeModule4-CM4, CM4IO:Raspberry-Pi-4-Compute-Module, symbol CM4IO:ComputeModule4-CM4
- added SW1: SW_Push, symbol Switch:SW_Push
- added SW3, SW4: SW_DPDT_x2, symbol Switch:SW_DPDT_x2
Connections:
- net +3.3V_PWR_1 is gone; now on net +3.3V_PWR: D2.2 (A)
- net +3.3V_PWR: now also IC5.5 (VCC), J3.1 (Pin_1), J3.17 (Pin_17), Module1.78 (GPIO_VREF(1.8v/3.3v_Input)), Module1.84 (+3.3v_(Output)), Module1.86 (+3.3v_(Output))
- net +5V_PWR: now also J3.2 (Pin_2), J3.4 (Pin_4), Module1.77 (+5v_(Input)), Module1.79 (+5v_(Input)), Module1.81 (+5v_(Input)), Module1.83 (+5v_(Input)), Module1.85 (+5v_(Input)), Module1.87 (+5v_(Input))
- net CAN_SPI_CLK: now also J3.23 (Pin_23), Module1.38 (GPIO11)
- net CAN_SPI_CS: now also J3.24 (Pin_24), Module1.39 (GPIO8)
- net CAN_SPI_MISO: now also J3.21 (Pin_21), Module1.40 (GPIO9)
- net CAN_SPI_MOSI: now also J3.19 (Pin_19), Module1.44 (GPIO10)
- net EEPROM_nWP: now also Module1.20 (EEPROM_nWP), SW4.2 (B)
- net GLOBAL_EN: now also Module1.99 (Global_EN)
- net GND: now also SW2.1, IC5.3 (GND), J3.14 (Pin_14), J3.20 (Pin_20), J3.25 (Pin_25), J3.30 (Pin_30), J3.34 (Pin_34), J3.39 (Pin_39), J3.6 (Pin_6), J3.9 (Pin_9), Module1.1 (GND), Module1.13 (GND), Module1.14 (GND), Module1.2 (GND), Module1.22 (GND), Module1.23 (GND), Module1.32 (GND), Module1.33 (GND), Module1.42 (GND), Module1.43 (GND), Module1.52 (GND), Module1.53 (GND), Module1.59 (GND), Module1.60 (GND), Module1.65 (GND), Module1.66 (GND), Module1.7 (GND), Module1.71 (GND), Module1.74 (GND), Module1.8 (GND), Module1.98 (GND), SW1.1, SW3.1 (A), SW3.4 (A), SW4.1 (A), SW4.6 (C)
- net GPIO13: now also J3.33 (Pin_33), Module1.28 (GPIO13)
- net GPIO14: now also J3.8 (Pin_8), Module1.55 (GPIO14)
- net GPIO15: now also J3.10 (Pin_10), Module1.51 (GPIO15)
- net GPIO16: now also J3.36 (Pin_36), Module1.29 (GPIO16)
- net GPIO17: now also J3.11 (Pin_11), Module1.50 (GPIO17)
- net GPIO18: now also J3.12 (Pin_12), Module1.49 (GPIO18)
- net GPIO19: now also J3.35 (Pin_35), Module1.26 (GPIO19)
- net GPIO2: now also J3.3 (Pin_3), Module1.58 (GPIO2)
- net GPIO20: now also J3.38 (Pin_38), Module1.27 (GPIO20)
- net GPIO21: now also J3.40 (Pin_40), Module1.25 (GPIO21)
- net GPIO22: now also J3.15 (Pin_15), Module1.46 (GPIO22)
- net GPIO23: now also J3.16 (Pin_16), Module1.47 (GPIO23)
- net GPIO24: now also J3.18 (Pin_18), Module1.45 (GPIO24)
- net GPIO25: now also J3.22 (Pin_22), Module1.41 (GPIO25)
- net GPIO26: now also J3.37 (Pin_37), Module1.24 (GPIO26)
- net GPIO27: now also J3.13 (Pin_13), Module1.48 (GPIO27)
- net GPIO3: now also J3.5 (Pin_5), Module1.56 (GPIO3)
- net GPIO4: now also J3.7 (Pin_7), Module1.54 (GPIO4)
- net GPIO5: now also J3.29 (Pin_29), Module1.34 (GPIO5)
- net GPIO6: now also J3.31 (Pin_31), Module1.30 (GPIO6)
- net GPIO7: now also J3.26 (Pin_26), Module1.37 (GPIO7)
- net RUN_PG: now also Module1.92 (RUN_PG), SW1.2
- net SCL0: now also Module1.80 (SCL0)
- net SDA0: now also Module1.82 (SDA0)
- net nEXTRST: now also Module1.100 (nEXTRST)
- net nPWR_LED: now also IC5.2 (A), Module1.95 (nPI_LED_PWR)
- net at R4.2: now also IC5.4
- net at R1.2: now also Module1.21 (PI_nLED_Activity)
- new net BT_Disable: Module1.91 (BT_nDisable), SW3.5 (B)
- new net CAN_INTR: J3.32 (Pin_32), Module1.31 (GPIO12)
- new net GPIO0: J3.27 (Pin_27), Module1.36 (ID_SD)
- new net GPIO1: J3.28 (Pin_28), Module1.35 (ID_SC)
- new net WiFi_Disable: Module1.89 (WiFi_nDisable), SW3.2 (B)
- new net nRPIBOOT: Module1.93 (nRPIBOOT), SW4.5 (B)
- no-connect marks 31 -> 35
Other:
- note added: "CM4 Reset Button"
- note added: "Full Reset Button"
- note added: "Press for >1 ms and then release to reset all 5V and 3.3V components."
- note added: "Press for >1 ms and then release to reset only the CM4 and any components connected to it (3.3V components)."
- note added: "Ready EMMC for flash"
- note added: "Wireless EN"
- note removed: "Disable wireless interfaces"
- note removed: "Not Fitted headers"
- note removed: "Pushing the button wakes the Raspberry Pi if it was previously in sleep but powered on. If the Pi is already awake, nothing happens."
- note removed: "Wake-up Button"
- moved on the sheet: D1, R1, SW2, TP1
