File: PWR_Distribution.kicad_sch (KiCad schematic)
At the start: 41 parts, among them U22 AP64501SP-13, U7 LM76202QPWPRQ1

Commit message: made more changes
Connections:
- net +12V is gone; now on net +12V_PWR: R44.1, U22.2 (VIN), U22.3 (EN)
- net +5V is gone; now on net +5V_PWR: R45.1
Changed lines of the file:
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@@
 	)
 	(junction
+		(at 111.76 124.46)
+		(diameter 0)
+		(color 0 0 0 0)
+	)
+	(junction
 		(at 60.96 120.65)
 		(diameter 0)
@@
 	)
 	(junction
-		(at 111.76 124.46)
-		(diameter 0)
-		(color 0 0 0 0)
-	)
-	(junction
 		(at 123.19 43.18)
 		(diameter 0)
@@
 	(wire
 		(pts
-			(xy 111.76 123.19) (xy 111.76 124.46)
-		)
-		(stroke
-			(width 0)
-			(type solid)
-		)
-	)
-	(wire
-		(pts
 			(xy 85.09 55.88) (xy 90.17 55.88)
 		)
@@
 	(wire
 		(pts
-			(xy 111.76 124.46) (xy 111.76 125.73)
+			(xy 111.76 123.19) (xy 111.76 124.46)
 		)
 		(stroke
@@
 	(wire
 		(pts
-			(xy 97.79 124.46) (xy 111.76 124.46)
-		)
-		(stroke
-			(width 0)
-			(type default)
-		)
-	)
-	(wire
-		(pts
 			(xy 242.57 53.34) (xy 242.57 52.07)
 		)
@@
 	(wire
 		(pts
+			(xy 105.41 124.46) (xy 111.76 124.46)
+		)
+		(stroke
+			(width 0)
+			(type default)
+		)
+	)
+	(wire
+		(pts
 			(xy 151.13 144.78) (xy 161.29 144.78)
 		)
@@
 	(wire
 		(pts
+			(xy 218.44 39.37) (xy 218.44 44.45)
+		)
+		(stroke
+			(width 0)
+			(type default)
+		)
+	)
+	(wire
+		(pts
 			(xy 133.35 109.22) (xy 133.35 120.65)
 		)
@@
 	(wire
 		(pts
-			(xy 218.44 40.64) (xy 218.44 44.45)
-		)
-		(stroke
-			(width 0)
-			(type default)
-		)
-	)
-	(wire
-		(pts
 			(xy 242.57 66.04) (xy 242.57 60.96)
 		)
@@
 	(wire
 		(pts
-			(xy 229.87 40.64) (xy 229.87 44.45)
+			(xy 229.87 39.37) (xy 229.87 44.45)
 		)
 		(stroke
@@
 	(wire
 		(pts
+			(xy 111.76 124.46) (xy 111.76 125.73)
+		)
+		(stroke
+			(width 0)
+			(type solid)
+		)
+	)
+	(wire
+		(pts
 			(xy 161.29 109.22) (xy 161.29 115.57)
 		)
@@
 	(hierarchical_label "+12V_PWR"
 		(shape input)
+		(at 218.44 39.37 90)
+		(fields_autoplaced yes)
+		(effects
+			(font
+				(size 1.27 1.27)
+			)
+			(justify left)
+		)
+	)
+	(hierarchical_label "+12V_PWR"
+		(shape input)
 		(at 62.23 114.3 0)
 		(fields_autoplaced yes)
@@
 		)
 	)
+	(hierarchical_label "+12V_PWR"
+		(shape input)
+		(at 105.41 124.46 180)
+		(fields_autoplaced yes)
+		(effects
+			(font
+				(size 1.27 1.27)
+			)
+			(justify right)
+		)
+	)
 	(hierarchical_label "+5V_PWR"
 		(shape output)
@@
 		)
 	)
+	(hierarchical_label "+5V_PWR"
+		(shape input)
+		(at 229.87 39.37 90)
+		(fields_autoplaced yes)
+		(effects
+			(font
+				(size 1.27 1.27)
+			)
+			(justify left)
+		)
+	)
 	(hierarchical_label "+12V_PWR"
 		(shape output)
@@
 	)
 	(symbol
-		(lib_id "power:+12V")
-		(at 218.44 40.64 0)
-		(unit 1)
-		(exclude_from_sim no)
-		(in_bom yes)
-		(on_board yes)
-		(dnp no)
-		(fields_autoplaced yes)
-		(property "Reference" "#PWR0108"
-			(at 218.44 44.45 0)
-			(effects
-				(font
-					(size 1.27 1.27)
-				)
-				(hide yes)
-			)
-		)
-		(property "Value" "+12V"
-			(at 218.44 36.83 0)
-			(effects
-				(font
-					(size 1.27 1.27)
-				)
-			)
-		)
-		(property "Footprint" ""
-			(at 218.44 40.64 0)
-			(effects
-				(font
-					(size 1.27 1.27)
-				)
-				(hide yes)
-			)
-		)
-		(property "Datasheet" ""
-			(at 218.44 40.64 0)
-			(effects
-				(font
-					(size 1.27 1.27)
-				)
-				(hide yes)
-			)
-		)
-		(property "Description" "Power symbol creates a global label with name \"+12V\""
-			(at 218.44 40.64 0)
-			(effects
-				(font
-					(size 1.27 1.27)
-				)
-				(hide yes)
-			)
-		)
-		(pin "1"
-		)
-		(instances
-			(project "PiBoard"
-				(path "/e4d65698-b8ec-4bf6-9f2b-a5010377155a/0c1fd794-8ba7-4f58-ad3e-1ee234c84a43"
-					(reference "#PWR0108")
-					(unit 1)
-				)
-			)
-		)
-	)
-	(symbol
 		(lib_id "Device:L")
 		(at 149.86 109.22 90)
@@
 	)
 	(symbol
-		(lib_id "power:+5V")
-		(at 229.87 40.64 0)
-		(unit 1)
-		(exclude_from_sim no)
-		(in_bom yes)
-		(on_board yes)
-		(dnp no)
-		(fields_autoplaced yes)
-		(property "Reference" "#PWR0112"
-			(at 229.87 44.45 0)
-			(effects
-				(font
-					(size 1.27 1.27)
-				)
-				(hide yes)
-			)
-		)
-		(property "Value" "+5V"
-			(at 229.87 35.56 0)
-			(effects
-				(font
-					(size 1.27 1.27)
-				)
-			)
-		)
-		(property "Footprint" ""
-			(at 229.87 40.64 0)
-			(effects
-				(font
-					(size 1.27 1.27)
-				)
-				(hide yes)
-			)
-		)
-		(property "Datasheet" ""
-			(at 229.87 40.64 0)
-			(effects
-				(font
-					(size 1.27 1.27)
-				)
-				(hide yes)
-			)
-		)
-		(property "Description" "Power symbol creates a global label with name \"+5V\""
-			(at 229.87 40.64 0)
-			(effects
-				(font
-					(size 1.27 1.27)
-				)
-				(hide yes)
-			)
-		)
-		(pin "1"
-		)
-		(instances
-			(project ""
-				(path "/e4d65698-b8ec-4bf6-9f2b-a5010377155a/0c1fd794-8ba7-4f58-ad3e-1ee234c84a43"
-					(reference "#PWR0112")
-					(unit 1)
-				)
-			)
-		)
-	)
-	(symbol
 		(lib_id "Device:C")
 		(at 190.5 113.03 0)
@@
 					(unit 1)
 				)
-			)
-		)
-	)
-	(symbol
-		(lib_id "power:+12V")
-		(at 97.79 124.46 0)
-		(unit 1)
-		(exclude_from_sim no)
-		(in_bom yes)
-		(on_board yes)
-		(dnp no)
-		(fields_autoplaced yes)
-		(property "Reference" "#PWR0119"
-			(at 97.79 128.27 0)
-			(effects
-				(font
-					(size 1.27 1.27)
-				)
-				(hide yes)
-			)
-		)
-		(property "Value" "+12V"
-			(at 97.79 119.38 0)
-			(effects
-				(font
-					(size 1.27 1.27)
-				)
-			)
-		)
-		(property "Footprint" ""
-			(at 97.79 124.46 0)
-			(effects
-				(font
-					(size 1.27 1.27)
-				)
-				(hide yes)
-			)
-		)
-		(property "Datasheet" ""
-			(at 97.79 124.46 0)
-			(effects
-				(font
-					(size 1.27 1.27)
-				)
-				(hide yes)
-			)
-		)
-		(property "Description" "Power symbol creates a global label with name \"+12V\""
-			(at 97.79 124.46 0)
-			(effects
-				(font
-					(size 1.27 1.27)
-				)
-				(hide yes)
-			)
-		)
-		(pin "1"
-		)
-		(instances
-			(project "PiBoard"
-				(path "/e4d65698-b8ec-4bf6-9f2b-a5010377155a/0c1fd794-8ba7-4f58-ad3e-1ee234c84a43"
-					(reference "#PWR0119")
-					(unit 1)
-				)

Commit message: finished USB i think, working on general gpio in more detail
Parts:
- added J1: CarPowerConnector, symbol utsvt-connectors:CarPowerConnector
Connections:
- net 12V_EXTN: no longer C14.1, D3.2 (A2), R7.1, U7.1 (IN_1), U7.2 (IN_2)
- new net: C14.1, D3.2 (A2), J1.1 (+12V), R7.1, U7.1 (IN_1), U7.2 (IN_2)
- new net GNDPWR: J1.2 (GND)
Other:
- moved on the sheet: D11, R46, TP10

Commit message: random stuff before i screw with my windows install
Connections:
- net 12V_EXTN is gone; now on net 12V_Extn: R46.1
- net 12V_Extn: now reaches C14.1, D3.2 (A2), J1.1 (+12V), R7.1, U7.1 (IN_1), U7.2 (IN_2)
Other:
- note added: "12V PWR"
- note added: "5V PWR"
- note added: "PWR FAULT"
- moved on the sheet: D11, D9, R44, R46, TP10

Commit message: we ballin??
Parts:
- removed C56, C57, C58, C59, C60, C61: 10u 35v, Capacitor_SMD:C_0805_2012Metric, symbol Device:C
- added C36, C37, C38, C39, C40, C41: 10u 35v, Capacitor_SMD:C_0805_2012Metric, symbol Device:C
- R43: value 10K -> 7.5K
Connections:
- net +12V_PWR: now also C36.1, C37.1, C38.1, C39.1, C40.1, C41.1
- net GND: now also C36.2, C37.2, C38.2, C39.2, C40.2, C41.2
Other:
- note added: "Current lim(A) = 12/Rilim(k) 1.7A = 12/7k ohms"
- note removed: "Current lim(A) = 12/Rilim(k) 1.2A = 12/10k ohms"
- moved on the sheet: C50, C62, C63, C64, C65, C66, C67, C68, C69, C70, L4, R47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
