File: USB_Ports.kicad_sch (KiCad schematic)
At the start: 28 parts, among them IC2 TPS2066TDGNRQ1, IC3 TPS2066TDGNRQ1, J10 3-2172091-2, J5 3-2172091-2, J6 3-2172091-2, J8 3-2172091-2

Commit message: we ballin??
Other:
- note added: "Current Limit Switches"
- note removed: "Current Limit switch"
Changed lines of the file:
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@@
 		)
 	)
-	(text "Current Limit switch"
+	(text "Current Limit Switches"
 		(exclude_from_sim no)
 		(at 87.884 25.908 0)
@@
 	(text "Current is limited to max 500mA per port."
 		(exclude_from_sim no)
-		(at 78.74 28.448 0)
+		(at 76.708 28.448 0)
 		(effects
 			(font
